File: Kicad_Design/PCB_ADS8694.sch (KiCad schematic (older format))
At the start: 1 part

Commit message: Se crea simbolo de ADS8694
Parts:
- removed U?: ADS8694, Package_SO:TSSOP-38_4.4x9.7mm_P0.5mm, symbol ads8694:ADS8694
- added U?: ADS8694, Package_SO:TSSOP-38_4.4x9.7mm_P0.5mm, symbol Analog_ADC:ADS8694
Changed lines of the file:
@@
 $EndDescr
 $Comp
-L ads8694:ADS8694 U?
-U 1 1 5CC9178D
-P 6050 3400
-F 0 "U?" H 6050 2011 50  0000 C CNN
-F 1 "ADS8694" H 6050 1920 50  0000 C CNN
-F 2 "Package_SO:TSSOP-38_4.4x9.7mm_P0.5mm" H 6050 3400 50  0001 C CNN
-F 3 "http://www.ti.com/lit/ds/symlink/ads8694.pdf" H 7000 4700 50  0001 C CNN
-	1    6050 3400
+L Analog_ADC:ADS8694 U?
+U 1 1 5CC8C75B
+P 5550 3900
+F 0 "U?" H 5550 2511 50  0000 C CNN
+F 1 "ADS8694" H 5550 2420 50  0000 C CNN
+F 2 "Package_SO:TSSOP-38_4.4x9.7mm_P0.5mm" H 5550 3900 50  0001 C CNN
+F 3 "http://www.ti.com/lit/ds/symlink/ads8694.pdf" H 6500 5200 50  0001 C CNN
+	1    5550 3900
 	1    0    0    -1
 $EndComp
