File: Kicad_Design/PCB_ADS8694/PCB_ADS8694.sch (KiCad schematic (older format))
At the start: 29 parts, among them J1 Conn_01x03_Male_Alimentación_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, J2 Conn_01x10_Female, J3 Conn_01x02_Male, J4 Conn_02x06_Male_Pmod_Spartan6, U1 LM7805_TO220, U2 AD8221, U3 AD8221, U4 ADS8694, U5 AD8221, U6 AD8221

Commit message: agregado de capacitores de desacoplo
Parts:
- removed C11: C, symbol Device:C
- removed C2, C4: 100nf, symbol Device:C
- added C12, C13, C21, C22, C23, C24: 100nf, Capacitor_THT:C_Disc_D5.0mm_W2.5mm_P5.00mm, symbol Device:C
- added C14, C16, C17, C18, C25, C26, C27, C28: 10uf, Capacitor_THT:CP_Radial_D4.0mm_P2.00mm, symbol Device:C
- added C15: 1uf, Capacitor_THT:C_Disc_D5.0mm_W2.5mm_P5.00mm, symbol Device:C
- added C19, C29: C, symbol Device:C
- added C?: 10uf, Capacitor_THT:C_Disc_D5.0mm_W2.5mm_P5.00mm, symbol Device:C
- C10, C9: value C -> 100nf; footprint (none) -> Capacitor_THT:C_Disc_D5.0mm_W2.5mm_P5.00mm
- C3, C5, C6, C7, C8: footprint (none) -> Capacitor_THT:CP_Radial_D4.0mm_P2.00mm
Connections:
- wire segments 72 -> 83
Other:
- moved on the sheet: C8, R1, RV1, RV2, RV3, RV4, U3

Commit message: Agregado de capacitores de desacople, cambios en simbolo de AD
Parts:
- removed C5: 10uF, Capacitor_THT:CP_Radial_D4.0mm_P2.00mm, symbol Device:CP
- removed C6: 1uF, Capacitor_THT:CP_Radial_D4.0mm_P2.00mm, symbol Device:CP
- removed C7: 22uF, Capacitor_THT:CP_Radial_D4.0mm_P2.00mm, symbol Device:CP
- removed J1: Conn_01x03_Male_Alimentación_analógica_externa_(+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, symbol Connector:Conn_01x03_Male
- removed J2: Conn_01x10_Female, symbol Connector:Conn_01x10_Female
- added C2, C6: 1uf, Capacitor_SMD:C_0603_1608Metric, symbol Device:C
- added C5: 10uf, Capacitor_SMD:C_0805_2012Metric, symbol Device:C
- added C7: 22uF, Capacitor_SMD:C_1206_3216Metric, symbol Device:C
- added J1: Screw_Terminal_01x03_Alimentación_analógica, TerminalBlock:TerminalBlock_Altech_AK300-3_P5.00mm, symbol Connector:Screw_Terminal_01x03
- added J2: Screw_Terminal_01x02_CH_AUX, TerminalBlock:TerminalBlock_Altech_AK300-2_P5.00mm, symbol Connector:Screw_Terminal_01x02
- added J5: Screw_Terminal_01x02_CH3, TerminalBlock:TerminalBlock_Altech_AK300-2_P5.00mm, symbol Connector:Screw_Terminal_01x02
- added J6: Screw_Terminal_01x02_CH2, TerminalBlock:TerminalBlock_Altech_AK300-2_P5.00mm, symbol Connector:Screw_Terminal_01x02
- added J7: Screw_Terminal_01x02_CH1, TerminalBlock:TerminalBlock_Altech_AK300-2_P5.00mm, symbol Connector:Screw_Terminal_01x02
- added J8: Screw_Terminal_01x02_CH0, TerminalBlock:TerminalBlock_Altech_AK300-2_P5.00mm, symbol Connector:Screw_Terminal_01x02
- C10, C12, C13, C21, C22, C23, C24, C9: footprint Capacitor_THT:C_Disc_D5.0mm_W2.5mm_P5.00mm -> Capacitor_SMD:C_0603_1608Metric
- C14, C16, C17, C18, C25, C26, C27, C28, C8: footprint Capacitor_THT:CP_Radial_D4.0mm_P2.00mm -> Capacitor_SMD:C_0805_2012Metric
- C15: footprint Capacitor_THT:C_Disc_D5.0mm_W2.5mm_P5.00mm -> Capacitor_SMD:C_0805_2012Metric
- C19, C29: footprint (none) -> Capacitor_SMD:C_0805_2012Metric
- C3: footprint Capacitor_THT:CP_Radial_D4.0mm_P2.00mm -> Capacitor_THT:C_Disc_D5.0mm_W2.5mm_P5.00mm
- C4: renamed from C?; footprint Capacitor_THT:C_Disc_D5.0mm_W2.5mm_P5.00mm -> Capacitor_SMD:C_0805_2012Metric
- J3: footprint (none) -> Connector_PinHeader_2.54mm:PinHeader_1x01_P2.54mm_Vertical
- J4: footprint (none) -> TerminalBlock:TerminalBlock_Altech_AK300-2_P5.00mm
- JP1: footprint (none) -> Connector_PinHeader_2.54mm:PinHeader_1x03_P2.54mm_Vertical
- R1, R2, R3: footprint (none) -> Resistor_THT:R_Axial_DIN0207_L6.3mm_D2.5mm_P10.16mm_Horizontal
- RV1, RV2, RV3, RV4: footprint (none) -> Potentiometer_THT:Potentiometer_Bourns_3266Y_Vertical
- U4: symbol Analog_ADC:ADS8694 -> PCB_ADS8694-rescue:ADS8694-Analog_ADC
Connections:
- wire segments 83 -> 92
Other:
- note added: "CONECTORES DE ENTRADA DE SEÑAL"
- note added: "ENTRADA CON ACONDICIONAMIENTO SIN FILTRO RC\n"
- note removed: "ENTRADA CON ACONDICIONAMIENTO SIN FILTRO RC, \nCON CAPACITOR PARA FILTRAR COMPONENTE DE CC"
- note removed: "ENTRADAS"
- moved on the sheet: C15

Commit message: Modificacion simbolo AD, agregado de capacitores de desacople, asignacion de huellas
Parts:
- U2, U3, U5, U6: footprint (none) -> Package_SO:MSOP-8_3x3mm_P0.65mm
Changed lines of the file:
@@
 F 0 "U3" H 2175 5472 60  0000 C CNN
 F 1 "AD8221" H 2175 5366 60  0000 C CNN
-F 2 "" H 2175 5075 50  0001 C CNN
+F 2 "Package_SO:MSOP-8_3x3mm_P0.65mm" H 2175 5075 50  0001 C CNN
 F 3 "" H 2175 5075 50  0001 C CNN
 	1    2175 5075
@@
 F 0 "U2" H 2275 7047 60  0000 C CNN
 F 1 "AD8221" H 2275 6941 60  0000 C CNN
-F 2 "" H 2275 6650 50  0001 C CNN
+F 2 "Package_SO:MSOP-8_3x3mm_P0.65mm" H 2275 6650 50  0001 C CNN
 F 3 "" H 2275 6650 50  0001 C CNN
 	1    2275 6650
@@
 F 0 "U6" H 8825 5972 60  0000 C CNN
 F 1 "AD8221" H 8825 5866 60  0000 C CNN
-F 2 "" H 8825 5575 50  0001 C CNN
+F 2 "Package_SO:MSOP-8_3x3mm_P0.65mm" H 8825 5575 50  0001 C CNN
 F 3 "" H 8825 5575 50  0001 C CNN
 	1    8825 5575
@@
 F 0 "U5" H 8700 3872 60  0000 C CNN
 F 1 "AD8221" H 8700 3766 60  0000 C CNN
-F 2 "" H 8700 3475 50  0001 C CNN
+F 2 "Package_SO:MSOP-8_3x3mm_P0.65mm" H 8700 3475 50  0001 C CNN
 F 3 "" H 8700 3475 50  0001 C CNN
 	1    8700 3475

Commit message: se elimina canal aux, se elimina jumper daisy
Parts:
- removed J2: Screw_Terminal_01x02_CH_AUX, TerminalBlock:TerminalBlock_Altech_AK300-2_P5.00mm, symbol Connector:Screw_Terminal_01x02
- removed J3: Conn_01x02_Male, Connector_PinHeader_2.54mm:PinHeader_1x01_P2.54mm_Vertical, symbol Connector:Conn_01x02_Male
- removed JP1: Jumper_3_Open, Connector_PinHeader_2.54mm:PinHeader_1x03_P2.54mm_Vertical, symbol Jumper:Jumper_3_Open
- C1: footprint Capacitor_THT:CP_Radial_D4.0mm_P2.00mm -> Capacitor_THT:CP_Radial_D5.0mm_P2.00mm
- C10, C9: value 100nf -> 100nf__CH1
- C12, C13: value 100nf -> 100nf_CH2
- C14, C16: value 10uf -> 10uf__CH1
- C17, C18: value 10uf -> 10uf_CH2
- C21, C22: value 100nf -> 100nf_CH0
- C23, C24: value 100nf -> 100nf_CH3
- C25, C26: value 10uf -> 10uf_CH0
- C27, C28: value 10uf -> 10uf_CH3
- J4: footprint TerminalBlock:TerminalBlock_Altech_AK300-2_P5.00mm -> Connector_PinHeader_2.54mm:PinHeader_2x06_P2.54mm_Horizontal
- U4: symbol PCB_ADS8694-rescue:ADS8694-Analog_ADC -> PCB_ADS8694-rescue:ADS8694-Analog_ADC-PCB_ADS8694-rescue
Connections:
- net labels removed: AUX_IN, DAISY
- wire segments 92 -> 88
- no-connect marks 2 -> 4
Other:
- note removed: "JUMPER PARA SELECCIONAR MODO DAISY-CHAIN"
- note removed: "PIN DAISY"
- note removed: "PIN SDO\n"

Commit message: Cambios en encapsulados. Agregado de serigrafía
Parts:
- C19, C29, C8: footprint Capacitor_SMD:C_0805_2012Metric -> Capacitor_THT:C_Disc_D5.0mm_W2.5mm_P5.00mm
- C7: footprint Capacitor_SMD:C_1206_3216Metric -> Capacitor_THT:CP_Radial_D5.0mm_P2.00mm
Changed lines of the file:
@@
 F 0 "C8" H 4015 5221 50  0000 L CNN
 F 1 "C" H 4015 5130 50  0000 L CNN
-F 2 "Capacitor_SMD:C_0805_2012Metric" H 3938 5025 50  0001 C CNN
+F 2 "Capacitor_THT:C_Disc_D5.0mm_W2.5mm_P5.00mm" H 3938 5025 50  0001 C CNN
 F 3 "~" H 3900 5175 50  0001 C CNN
 	1    3900 5175
@@
 F 0 "C19" H 4115 6796 50  0000 L CNN
 F 1 "C" H 4115 6705 50  0000 L CNN
-F 2 "Capacitor_SMD:C_0805_2012Metric" H 4038 6600 50  0001 C CNN
+F 2 "Capacitor_THT:C_Disc_D5.0mm_W2.5mm_P5.00mm" H 4038 6600 50  0001 C CNN
 F 3 "~" H 4000 6750 50  0001 C CNN
 	1    4000 6750
@@
 F 0 "C29" H 10665 5721 50  0000 L CNN
 F 1 "C" H 10665 5630 50  0000 L CNN
-F 2 "Capacitor_SMD:C_0805_2012Metric" H 10588 5525 50  0001 C CNN
+F 2 "Capacitor_THT:C_Disc_D5.0mm_W2.5mm_P5.00mm" H 10588 5525 50  0001 C CNN
 F 3 "~" H 10550 5675 50  0001 C CNN
 	1    10550 5675
@@
 F 0 "C7" V 7300 2000 50  0000 L CNN
 F 1 "22uF" V 7475 1925 50  0000 L CNN
-F 2 "Capacitor_SMD:C_1206_3216Metric" H 7388 1800 50  0001 C CNN
+F 2 "Capacitor_THT:CP_Radial_D5.0mm_P2.00mm" H 7388 1800 50  0001 C CNN
 F 3 "~" H 7350 1950 50  0001 C CNN
 	1    7350 1950

Commit message: PCB V1
Parts:
- removed U4: ADS8694, Package_SO:TSSOP-38_4.4x9.7mm_P0.5mm, symbol PCB_ADS8694-rescue:ADS8694-Analog_ADC-PCB_ADS8694-rescue
- added U4: ADS8694_Vers2, Package_SO:TSSOP-38_4.4x9.7mm_P0.5mm, symbol ads8694_vers2:ADS8694_Vers2
Changed lines of the file:
@@
 EESchema Schematic File Version 4
-LIBS:PCB_ADS8694-cache
 EELAYER 29 0
 EELAYER END
@@
 F 3 "~" H 4950 1850 50  0001 C CNN
 	1    4950 1850
-	1    0    0    -1
-$EndComp
-$Comp
-L PCB_ADS8694-rescue:ADS8694-Analog_ADC-PCB_ADS8694-rescue U4
-U 1 1 5CCB2EF2
-P 5750 4500
-F 0 "U4" H 5750 4550 50  0000 C CNN
-F 1 "ADS8694" H 5750 4450 50  0000 C CNN
-F 2 "Package_SO:TSSOP-38_4.4x9.7mm_P0.5mm" H 5750 4500 50  0001 C CNN
-F 3 "http://www.ti.com/lit/ds/symlink/ads8694.pdf" H 6700 5800 50  0001 C CNN
-	1    5750 4500
 	1    0    0    -1
 $EndComp
@@
 L power:GNDD #PWR0119
 U 1 1 5CD863F9
-P 6100 5800
-F 0 "#PWR0119" H 6100 5550 50  0001 C CNN
-F 1 "GNDD" H 6104 5645 50  0000 C CNN
-F 2 "" H 6100 5800 50  0001 C CNN
-F 3 "" H 6100 5800 50  0001 C CNN
-	1    6100 5800
+P 6050 5800
+F 0 "#PWR0119" H 6050 5550 50  0001 C CNN
+F 1 "GNDD" H 6054 5645 50  0000 C CNN
+F 2 "" H 6050 5800 50  0001 C CNN
+F 3 "" H 6050 5800 50  0001 C CNN
+	1    6050 5800
 	1    0    0    -1
 $EndComp
@@
 Text GLabel 5750 3100 1    50   Input ~ 0
 AVDD
-Wire Wire Line
-	5650 5800 5650 5875
-Wire Wire Line
-	5450 5875 5450 5800
-Wire Wire Line
-	5550 5800 5550 5875
-Connection ~ 5550 5875
-Wire Wire Line
-	5550 5875 5450 5875
 $Comp
 L power:GNDA #PWR034
 U 1 1 5CEF30B1
-P 5650 5875
-F 0 "#PWR034" H 5650 5625 50  0001 C CNN
-F 1 "GNDA" H 5655 5702 50  0000 C CNN
-F 2 "" H 5650 5875 50  0001 C CNN
-F 3 "" H 5650 5875 50  0001 C CNN
-	1    5650 5875
-	1    0    0    -1
-$EndComp
-Wire Wire Line
-	5750 5800 5750 5875
-Wire Wire Line
-	5750 5875 5650 5875
-Connection ~ 5650 5875
-Wire Wire Line
-	5850 5800 5850 5875
-Wire Wire Line
-	5850 5875 5750 5875
-Connection ~ 5750 5875
-Wire Wire Line
-	5550 5875 5650 5875
+P 5600 5900
+F 0 "#PWR034" H 5600 5650 50  0001 C CNN
+F 1 "GNDA" H 5605 5727 50  0000 C CNN
+F 2 "" H 5600 5900 50  0001 C CNN
+F 3 "" H 5600 5900 50  0001 C CNN
+	1    5600 5900
+	1    0    0    -1
+$EndComp
 $Comp
 L Device:C C7
@@
 Text GLabel 4750 1750 0    50   Input ~ 0
 CS
+$Comp
+L ads8694_vers2:ADS8694_Vers2 U4
+U 1 1 5CE32CBF
+P 5750 4500
+F 0 "U4" H 5750 5981 50  0000 C CNN
+F 1 "ADS8694_Vers2" H 5750 5890 50  0000 C CNN
+F 2 "Package_SO:TSSOP-38_4.4x9.7mm_P0.5mm" H 5750 4500 50  0001 C CNN
+F 3 "http://www.ti.com/lit/ds/symlink/ads8694.pdf" H 6700 5800 50  0001 C CNN
+	1    5750 4500
+	1    0    0    -1
+$EndComp
+Wire Wire Line
+	5400 5800 5400 5900
+Wire Wire Line
+	5400 5900 5500 5900
+Wire Wire Line
+	5500 5800 5500 5900
+Connection ~ 5500 5900
+Wire Wire Line
+	5500 5900 5600 5900
+Wire Wire Line
+	5600 5800 5600 5900
+Connection ~ 5600 5900
+Wire Wire Line
+	5700 5800 5700 5900
+Wire Wire Line
+	5700 5900 5625 5900
+Wire Wire Line
+	5800 5800 5800 5900
+Wire Wire Line
+	5800 5900 5700 5900
+Connection ~ 5700 5900
 $EndSCHEMATC

Commit message: PCB V1
Other:
- note removed: "COMUNICACIÓN SPI\nFunción de pines Pmod:\n1: SCLK\n2: SDI -> Se conecta con SDO de AD8694\n3: SDO -> Se conecta con SDI de AD8694\n4: /CS (Activo por bajo)\n7: /RST-/PD (Activo por bajo)\n8: ALARM (Entrada; activo por alto)"
- moved on the sheet: J4
Changed lines of the file:
@@
 L Connector_Generic:Conn_02x06_Top_Bottom J4
 U 1 1 5CCB59D8
-P 4950 1850
-F 0 "J4" H 5000 2267 50  0000 C CNN
-F 1 "Conn_02x06_Male_Pmod_Spartan6" H 5000 2176 50  0000 C CNN
-F 2 "Connector_PinHeader_2.54mm:PinHeader_2x06_P2.54mm_Horizontal" H 4950 1850 50  0001 C CNN
-F 3 "~" H 4950 1850 50  0001 C CNN
-	1    4950 1850
+P 5100 1175
+F 0 "J4" H 5150 1592 50  0000 C CNN
+F 1 "Conn_02x06_Male_Pmod_Spartan6" H 5150 1501 50  0000 C CNN
+F 2 "Connector_PinHeader_2.54mm:PinHeader_2x06_P2.54mm_Horizontal" H 5100 1175 50  0001 C CNN
+F 3 "~" H 5100 1175 50  0001 C CNN
+	1    5100 1175
 	1    0    0    -1
 $EndComp
@@
 Wire Wire Line
 	2500 1000 2500 1050
-Text GLabel 6250 4400 2    50   Input ~ 0
+Text GLabel 6250 4400 2    50   Input ~ 6
 REFSEL
-Text GLabel 6250 4700 2    50   Input ~ 0
+Text GLabel 6250 4700 2    50   Input ~ 6
 ALARM
-Text GLabel 6250 4900 2    50   Input ~ 0
+Text GLabel 6250 4900 2    50   Input ~ 6
 REFCAP
-Text GLabel 6250 5100 2    50   Input ~ 0
+Text GLabel 6250 5100 2    50   Input ~ 6
 REFIO
-Text GLabel 6250 4200 2    50   Input ~ 0
+Text GLabel 6250 4200 2    50   Input ~ 6
 RST-PD
-Text GLabel 6250 3900 2    50   Input ~ 0
+Text GLabel 6250 3900 2    50   Input ~ 6
 CS
-Text GLabel 6250 3800 2    50   Input ~ 0
+Text GLabel 6250 3800 2    50   Input ~ 6
 SCLK
-Text GLabel 6250 3700 2    50   Input ~ 0
+Text GLabel 6250 3700 2    50   Input ~ 6
 SDI
-Text GLabel 6250 3600 2    50   Input ~ 0
+Text GLabel 6250 3600 2    50   Input ~ 6
 SDO
-Text GLabel 5250 3800 0    50   Input ~ 0
+Text GLabel 5250 3800 0    50   Input ~ 6
 AIN_1P
-Text GLabel 5250 4000 0    50   Input ~ 0
+Text GLabel 5250 4000 0    50   Input ~ 6
 AIN_2P
-Text GLabel 5250 4200 0    50   Input ~ 0
+Text GLabel 5250 4200 0    50   Input ~ 6
 AIN_3P
-Text GLabel 7200 800  0    50   Input ~ 0
+Text GLabel 7200 800  0    50   Input ~ 6
 REFSEL
-Text GLabel 7200 1150 0    50   Input ~ 0
+Text GLabel 7200 1150 0    50   Input ~ 6
 REFIO
-Text GLabel 7200 1550 0    50   Input ~ 0
+Text GLabel 7200 1550 0    50   Input ~ 6
 REFCAP
 Wire Wire Line
 	7200 1550 7200 1950
-Text Notes 6750 2650 0    50   ~ 0
+Text Notes 6750 2650 0    50   ~ 6
 CONFIGURACIÓN PARA USAR\nREFERENCIA INTERNA 4.096 [V]\n
-Text Notes 4800 2350 0    50   ~ 0
+Text Notes 4950 1675 0    50   ~ 6
 PMOD FPGA
 Wire Notes Line
@@
 Wire Notes Line
 	2950 650  950  650
-Text Notes 1450 1750 0    50   ~ 0
+Text Notes 1450 1750 0    50   ~ 6
 REGULADOR DE TENSIÓN, 5V\n
-Text Notes 7450 7500 0    79   ~ 0
+Text Notes 7450 7500 0    79   ~ 6
 PCB ADC8694
 Wire Notes Line
 	950  650  950  1800
-Text GLabel 4750 1950 0    50   Input ~ 0
+Text GLabel 4900 1275 0    50   Input ~ 6
 SCLK
-Text GLabel 4750 2150 0    50   Input ~ 0
+Text GLabel 4900 1475 0    50   Input ~ 6
 SDO
-Text GLabel 4750 1850 0    50   Input ~ 0
+Text GLabel 4900 1175 0    50   Input ~ 6
 SDI
-Text Notes 4450 1350 0    50   ~ 0
-COMUNICACIÓN SPI\nFunción de pines Pmod:\n1: SCLK\n2: SDI -> Se conecta con SDO de AD8694\n3: SDO -> Se conecta con SDI de AD8694\n4: /CS (Activo por bajo)\n7: /RST-/PD (Activo por bajo)\n8: ALARM (Entrada; activo por alto)
-Wire Notes Line
-	4150 2450 6200 2450
-Wire Notes Line
-	6200 2450 6200 650
 Wire Notes Line
 	6200 650  4150 650
-Text Notes 1400 2700 0    50   ~ 0
+Text Notes 1400 2700 0    50   ~ 6
 FUENTE DE CC EXTERNA, +-VCC
 Wire Notes Line
@@
 Wire Wire Line
 	5250 3700 4600 3700
-NoConn ~ 4750 2050
-NoConn ~ 5250 1650
+NoConn ~ 4900 1375
+NoConn ~ 5400 975
 $Comp
 L power:GNDD #PWR0118
 U 1 1 5CD843B0
-P 5525 1850
-F 0 "#PWR0118" H 5525 1600 50  0001 C CNN
-F 1 "GNDD" H 5529 1695 50  0000 C CNN
-F 2 "" H 5525 1850 50  0001 C CNN
-F 3 "" H 5525 1850 50  0001 C CNN
-	1    5525 1850
+P 5675 1175
+F 0 "#PWR0118" H 5675 925 50  0001 C CNN
+F 1 "GNDD" H 5679 1020 50  0000 C CNN
+F 2 "" H 5675 1175 50  0001 C CNN
+F 3 "" H 5675 1175 50  0001 C CNN
+	1    5675 1175
 	1    0    0    -1
 $EndComp
@@
 	1    0    0    -1
 $EndComp
-Text GLabel 9200 3425 2    50   Input ~ 0
+Text GLabel 9200 3425 2    50   Input ~ 6
 AIN_0P
-Text GLabel 8200 3625 0    50   Input ~ 0
+Text GLabel 8200 3625 0    50   Input ~ 6
 AIN_0+
-Text GLabel 8200 3325 0    50   Input ~ 0
+Text GLabel 8200 3325 0    50   Input ~ 6
 AIN_0-
 $Comp
@@
 	0    1    1    0
 $EndComp
-Text GLabel 8325 5425 0    50   Input ~ 0
+Text GLabel 8325 5425 0    50   Input ~ 6
 AIN_3-
-Text GLabel 8325 5725 0    50   Input ~ 0
+Text GLabel 8325 5725 0    50   Input ~ 6
 AIN_3+
 Connection ~ 1125 6750
@@
 	0    1    1    0
 $EndComp
-Text GLabel 1775 6500 0    50   Input ~ 0
+Text GLabel 1775 6500 0    50   Input ~ 6
 AIN_2-
-Text GLabel 1775 6800 0    50   Input ~ 0
+Text GLabel 1775 6800 0    50   Input ~ 6
 AIN_2+
 Connection ~ 1025 5175
@@
 	0    1    1    0
 $EndComp
-Text GLabel 1675 4925 0    50   Input ~ 0
+Text GLabel 1675 4925 0    50   Input ~ 6
 AIN_1-
-Text GLabel 1675 5225 0    50   Input ~ 0
+Text GLabel 1675 5225 0    50   Input ~ 6
 AIN_1+
 $Comp
@@
 	1    0    0    -1
 $EndComp
-Text Notes 8100 4375 0    50   ~ 0
+Text Notes 8100 4375 0    50   ~ 6
 ENTRADA CON ACONDICIONAMIENTO SIN FILTRO RC\n
-Text Notes 1275 4175 0    50   ~ 0
+Text Notes 1275 4175 0    50   ~ 6
 CONECTORES DE ENTRADA DE SEÑAL
 $Comp
 L power:VDD #PWR0112
 U 1 1 5CD79A34
-P 5250 2050
-F 0 "#PWR0112" H 5250 1900 50  0001 C CNN
-F 1 "VDD" V 5268 2177 50  0000 L CNN
-F 2 "" H 5250 2050 50  0001 C CNN
-F 3 "" H 5250 2050 50  0001 C CNN
-	1    5250 2050
+P 5400 1375
+F 0 "#PWR0112" H 5400 1225 50  0001 C CNN
+F 1 "VDD" V 5418 1502 50  0000 L CNN
+F 2 "" H 5400 1375 50  0001 C CNN
+F 3 "" H 5400 1375 50  0001 C CNN
+	1    5400 1375
 	0    1    1    0
 $EndComp
@@
 L power:VDD #PWR0116
 U 1 1 5CD7F938
-P 5250 2150
-F 0 "#PWR0116" H 5250 2000 50  0001 C CNN
-F 1 "VDD" V 5267 2278 50  0000 L CNN
-F 2 "" H 5250 2150 50  0001 C CNN
-F 3 "" H 5250 2150 50  0001 C CNN
-	1    5250 2150
+P 5400 1475
+F 0 "#PWR0116" H 5400 1325 50  0001 C CNN
+F 1 "VDD" V 5417 1603 50  0000 L CNN
+F 2 "" H 5400 1475 50  0001 C CNN
+F 3 "" H 5400 1475 50  0001 C CNN
+	1    5400 1475
 	0    1    1    0
 $EndComp
@@
 	1    0    0    -1
 $EndComp
-Text GLabel 2500 1000 2    50   Input ~ 0
+Text GLabel 2500 1000 2    50   Input ~ 6
 AVDD
-Text GLabel 5650 3100 1    50   Input ~ 0
+Text GLabel 5650 3100 1    50   Input ~ 6
 AVDD
 $Comp
@@
 Wire Wire Line
 	4600 3700 4600 3900
-Text GLabel 5250 3600 0    50   Input ~ 0
+Text GLabel 5250 3600 0    50   Input ~ 6
 AIN_0P
 $Comp
@@
 	0    1    1    0
 $EndComp
-Text GLabel 3900 5025 2    50   Input ~ 0
+Text GLabel 3900 5025 2    50   Input ~ 6
 AIN_1P
 $Comp
@@
 	0    1    1    0
 $EndComp
-Text GLabel 4000 6600 2    50   Input ~ 0
+Text GLabel 4000 6600 2    50   Input ~ 6
 AIN_2P
 $Comp
@@
 	0    1    1    0
 $EndComp
-Text GLabel 10550 5525 2    50   Input ~ 0
+Text GLabel 10550 5525 2    50   Input ~ 6
 AIN_3P
 $Comp
@@
 	1    0    0    -1
 $EndComp
-Text GLabel 5750 3100 1    50   Input ~ 0
+Text GLabel 5750 3100 1    50   Input ~ 6
 AVDD
 $Comp
@@
 	-1   0    0    1
 $EndComp
-Text GLabel 3950 3050 1    50   Input ~ 0
+Text GLabel 3950 3050 1    50   Input ~ 6
 AVDD
 Wire Wire Line
@@
 Wire Notes Line
 	1250 2850 1250 4225
-Text GLabel 1850 3225 2    50   Input ~ 0
+Text GLabel 1850 3225 2    50   Input ~ 6
 AIN_3+
-Text GLabel 1850 3325 2    50   Input ~ 0
+Text GLabel 1850 3325 2    50   Input ~ 6
 AIN_3-
-Text GLabel 1850 3450 2    50   Input ~ 0
+Text GLabel 1850 3450 2    50   Input ~ 6
 AIN_2+
-Text GLabel 1850 3550 2    50   Input ~ 0
+Text GLabel 1850 3550 2    50   Input ~ 6
 AIN_2-
-Text GLabel 1850 3675 2    50   Input ~ 0
+Text GLabel 1850 3675 2    50   Input ~ 6
 AIN_1+
-Text GLabel 1850 3775 2    50   Input ~ 0
+Text GLabel 1850 3775 2    50   Input ~ 6
 AIN_1-
-Text GLabel 1850 3900 2    50   Input ~ 0
+Text GLabel 1850 3900 2    50   Input ~ 6
 AIN_0+
-Text GLabel 1850 4000 2    50   Input ~ 0
+Text GLabel 1850 4000 2    50   Input ~ 6
 AIN_0-
-Text Notes 1475 7575 0    50   ~ 0
+Text Notes 1475 7575 0    50   ~ 6
 ACONDICIONAMIENTO CON FILTRO PASA BAJO RC
 Wire Notes Line
@@
 NoConn ~ 5250 5300
 Wire Wire Line
-	5250 1850 5350 1850
-Wire Wire Line
-	5250 1950 5350 1950
-Wire Wire Line
-	5350 1950 5350 1850
-Connection ~ 5350 1850
-Wire Wire Line
-	5350 1850 5525 1850
-Wire Notes Line
-	4150 650  4150 2450
+	5400 1175 5500 1175
+Wire Wire Line
+	5400 1275 5500 1275
+Wire Wire Line
+	5500 1275 5500 1175
+Connection ~ 5500 1175
+Wire Wire Line
+	5500 1175 5675 1175
 $Comp
 L power:GNDD #PWR0106
@@
 Wire Wire Line
 	6825 4000 6250 4000
-Text GLabel 4750 1650 0    50   Input ~ 0
+Text GLabel 4900 975  0    50   Input ~ 6
 RST-PD
-Text GLabel 5250 1750 2    50   Input ~ 0
+Text GLabel 5400 1075 2    50   Input ~ 6
 ALARM
-Text GLabel 4750 1750 0    50   Input ~ 0
+Text GLabel 4900 1075 0    50   Input ~ 6
 CS
 $Comp
@@
 	5800 5900 5700 5900
 Connection ~ 5700 5900
+Wire Notes Line
+	4150 650  4150 1750
+Wire Notes Line
+	4150 1750 6200 1750
+Wire Notes Line
+	6200 1750 6200 650
 $EndSCHEMATC
