File: Kicad_Design/PCB_ADS8694/PCB_ADS8694.sch (KiCad schematic (older format))
At the start: 46 parts, among them J1 Screw_Terminal_01x03_Alimenta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, J4 Conn_02x06_Male_Pmod_Spartan6, J5 Screw_Terminal_01x02_CH3, J6 Screw_Terminal_01x02_CH2, J7 Screw_Terminal_01x02_CH1, J8 Screw_Terminal_01x02_CH0, U1 LM7805_TO220, U2 AD8221, U3 AD8221, U4 ADS8694_Vers2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

Commit message: Cambios en conector pmod
Connections:
- net ALARM: now also J4.5 (Pin_5); no longer J4.8 (Pin_8)
- net CS: now also J4.11 (Pin_11); no longer J4.2 (Pin_2)
- net GNDA: now also U4.32 (AGND), U4.8 (AGND); no longer C4.1, J4.10 (Pin_10), J4.9 (Pin_9), U4.3 (DAISY), U4.33 (DGND)
- net RST-PD: now also J4.12 (Pin_12); no longer J4.1 (Pin_1)
- net SCLK: now also J4.9 (Pin_9); no longer J4.4 (Pin_4)
- net SDI: now also J4.10 (Pin_10); no longer J4.3 (Pin_3)
- net SDO: now also J4.7 (Pin_7); no longer J4.6 (Pin_6)
- net VDD: now also J4.1 (Pin_1), J4.2 (Pin_2); no longer J4.11 (Pin_11), J4.12 (Pin_12)
- new net GNDD: C4.1, J4.3 (Pin_3), J4.4 (Pin_4), U4.3 (DAISY), U4.33 (DGND)
Changed lines of the file:
@@
 Wire Notes Line
 	950  650  950  1800
-Text GLabel 4900 1275 0    50   Input ~ 10
+Text GLabel 5400 1175 2    50   Input ~ 10
 SCLK
-Text GLabel 4900 1475 0    50   Input ~ 10
+Text GLabel 5400 975  2    50   Input ~ 10
 SDO
-Text GLabel 4900 1175 0    50   Input ~ 10
+Text GLabel 5400 1275 2    50   Input ~ 10
 SDI
 Wire Notes Line
@@
 Wire Wire Line
 	5250 3700 4600 3700
-NoConn ~ 4900 1375
-NoConn ~ 5400 975
+NoConn ~ 4900 1475
+NoConn ~ 5400 1075
 $Comp
 L power:GNDD #PWR0118
 U 1 1 5CD843B0
-P 5675 1175
-F 0 "#PWR0118" H 5675 925 50  0001 C CNN
-F 1 "GNDD" H 5679 1020 50  0000 C CNN
-F 2 "" H 5675 1175 50  0001 C CNN
-F 3 "" H 5675 1175 50  0001 C CNN
-	1    5675 1175
+P 4475 1200
+F 0 "#PWR0118" H 4475 950 50  0001 C CNN
+F 1 "GNDD" H 4479 1045 50  0000 C CNN
+F 2 "" H 4475 1200 50  0001 C CNN
+F 3 "" H 4475 1200 50  0001 C CNN
+	1    4475 1200
 	1    0    0    -1
 $EndComp
@@
 L power:VDD #PWR0112
 U 1 1 5CD79A34
-P 5400 1375
-F 0 "#PWR0112" H 5400 1225 50  0001 C CNN
-F 1 "VDD" V 5418 1502 50  0000 L CNN
-F 2 "" H 5400 1375 50  0001 C CNN
-F 3 "" H 5400 1375 50  0001 C CNN
-	1    5400 1375
-	0    1    1    0
+P 4900 975
+F 0 "#PWR0112" H 4900 825 50  0001 C CNN
+F 1 "VDD" V 4918 1102 50  0000 L CNN
+F 2 "" H 4900 975 50  0001 C CNN
+F 3 "" H 4900 975 50  0001 C CNN
+	1    4900 975
+	0    -1   -1   0
 $EndComp
 $Comp
 L power:VDD #PWR0116
 U 1 1 5CD7F938
-P 5400 1475
-F 0 "#PWR0116" H 5400 1325 50  0001 C CNN
-F 1 "VDD" V 5417 1603 50  0000 L CNN
-F 2 "" H 5400 1475 50  0001 C CNN
-F 3 "" H 5400 1475 50  0001 C CNN
-	1    5400 1475
-	0    1    1    0
+P 4900 1075
+F 0 "#PWR0116" H 4900 925 50  0001 C CNN
+F 1 "VDD" V 4917 1203 50  0000 L CNN
+F 2 "" H 4900 1075 50  0001 C CNN
+F 3 "" H 4900 1075 50  0001 C CNN
+	1    4900 1075
+	0    -1   -1   0
 $EndComp
 $Comp
@@
 NoConn ~ 5250 5400
 NoConn ~ 5250 5300
-Wire Wire Line
-	5400 1175 5500 1175
-Wire Wire Line
-	5400 1275 5500 1275
-Wire Wire Line
-	5500 1275 5500 1175
-Connection ~ 5500 1175
-Wire Wire Line
-	5500 1175 5675 1175
 $Comp
 L power:GNDD #PWR0106
@@
 Wire Wire Line
 	6825 4000 6250 4000
-Text GLabel 4900 975  0    50   Input ~ 10
+Text GLabel 5400 1475 2    50   Input ~ 10
 RST-PD
-Text GLabel 5400 1075 2    50   Input ~ 10
+Text GLabel 4900 1375 0    50   Input ~ 10
 ALARM
-Text GLabel 4900 1075 0    50   Input ~ 10
+Text GLabel 5400 1375 2    50   Input ~ 10
 CS
 $Comp
@@
 	5700 5800 5700 5900
 Wire Wire Line
-	5700 5900 5625 5900
-Wire Wire Line
 	5800 5800 5800 5900
 Wire Wire Line
 	5800 5900 5700 5900
+Wire Notes Line
+	4150 650  4150 1750
+Wire Notes Line
+	4150 1750 6200 1750
+Wire Notes Line
+	6200 1750 6200 650
+Wire Wire Line
+	5600 5900 5700 5900
 Connection ~ 5700 5900
-Wire Notes Line
-	4150 650  4150 1750
-Wire Notes Line
-	4150 1750 6200 1750
-Wire Notes Line
-	6200 1750 6200 650
-$Comp
-L power:GNDA #PWR01
-U 1 1 5CE84135
-P 8275 6825
-F 0 "#PWR01" H 8275 6575 50  0001 C CNN
-F 1 "GNDA" H 8280 6652 50  0000 C CNN
-F 2 "" H 8275 6825 50  0001 C CNN
-F 3 "" H 8275 6825 50  0001 C CNN
-	1    8275 6825
-	1    0    0    -1
-$EndComp
-$Comp
-L power:GNDD #PWR07
-U 1 1 5CE84736
-P 8650 6825
-F 0 "#PWR07" H 8650 6575 50  0001 C CNN
-F 1 "GNDD" H 8654 6670 50  0000 C CNN
-F 2 "" H 8650 6825 50  0001 C CNN
-F 3 "" H 8650 6825 50  0001 C CNN
-	1    8650 6825
-	1    0    0    -1
-$EndComp
-Wire Wire Line
-	8275 6825 8275 6775
-Wire Wire Line
-	8275 6775 8650 6775
-Wire Wire Line
-	8650 6775 8650 6825
+Wire Wire Line
+	4900 1275 4825 1275
+Wire Wire Line
+	4825 1275 4825 1175
+Connection ~ 4825 1175
+Wire Wire Line
+	4825 1175 4900 1175
+Wire Wire Line
+	4475 1200 4475 1175
+Wire Wire Line
+	4475 1175 4825 1175
 $EndSCHEMATC

Commit message: Capacitores 10uF de smd a THT
Parts:
- C14, C16, C17, C18, C25, C26, C27, C28, C4, C5: footprint Capacitor_SMD:C_0805_2012Metric -> Capacitor_THT:CP_Radial_D5.0mm_P2.00mm
Changed lines of the file:
@@
 F 0 "C14" H 3265 4821 50  0000 L CNN
 F 1 "10uf__CH1" H 3250 4700 50  0000 L CNN
-F 2 "Capacitor_SMD:C_0805_2012Metric" H 3188 4625 50  0001 C CNN
+F 2 "Capacitor_THT:CP_Radial_D5.0mm_P2.00mm" H 3188 4625 50  0001 C CNN
 F 3 "~" H 3150 4775 50  0001 C CNN
 	1    3150 4775
@@
 F 0 "C16" H 3265 5421 50  0000 L CNN
 F 1 "10uf__CH1" H 3175 5250 50  0000 L CNN
-F 2 "Capacitor_SMD:C_0805_2012Metric" H 3188 5225 50  0001 C CNN
+F 2 "Capacitor_THT:CP_Radial_D5.0mm_P2.00mm" H 3188 5225 50  0001 C CNN
 F 3 "~" H 3150 5375 50  0001 C CNN
 	1    3150 5375
@@
 F 0 "C17" H 3365 6396 50  0000 L CNN
 F 1 "10uf_CH2" H 3325 6275 50  0000 L CNN
-F 2 "Capacitor_SMD:C_0805_2012Metric" H 3288 6200 50  0001 C CNN
+F 2 "Capacitor_THT:CP_Radial_D5.0mm_P2.00mm" H 3288 6200 50  0001 C CNN
 F 3 "~" H 3250 6350 50  0001 C CNN
 	1    3250 6350
@@
 F 0 "C18" H 3365 6996 50  0000 L CNN
 F 1 "10uf_CH2" H 3300 6850 50  0000 L CNN
-F 2 "Capacitor_SMD:C_0805_2012Metric" H 3288 6800 50  0001 C CNN
+F 2 "Capacitor_THT:CP_Radial_D5.0mm_P2.00mm" H 3288 6800 50  0001 C CNN
 F 3 "~" H 3250 6950 50  0001 C CNN
 	1    3250 6950
@@
 F 0 "C27" H 9915 5321 50  0000 L CNN
 F 1 "10uf_CH3" H 9850 5200 50  0000 L CNN
-F 2 "Capacitor_SMD:C_0805_2012Metric" H 9838 5125 50  0001 C CNN
+F 2 "Capacitor_THT:CP_Radial_D5.0mm_P2.00mm" H 9838 5125 50  0001 C CNN
 F 3 "~" H 9800 5275 50  0001 C CNN
 	1    9800 5275
@@
 F 0 "C28" H 9915 5921 50  0000 L CNN
 F 1 "10uf_CH3" H 9850 5750 50  0000 L CNN
-F 2 "Capacitor_SMD:C_0805_2012Metric" H 9838 5725 50  0001 C CNN
+F 2 "Capacitor_THT:CP_Radial_D5.0mm_P2.00mm" H 9838 5725 50  0001 C CNN
 F 3 "~" H 9800 5875 50  0001 C CNN
 	1    9800 5875
@@
 F 0 "C25" H 9790 3221 50  0000 L CNN
 F 1 "10uf_CH0" H 9775 3100 50  0000 L CNN
-F 2 "Capacitor_SMD:C_0805_2012Metric" H 9713 3025 50  0001 C CNN
+F 2 "Capacitor_THT:CP_Radial_D5.0mm_P2.00mm" H 9713 3025 50  0001 C CNN
 F 3 "~" H 9675 3175 50  0001 C CNN
 	1    9675 3175
@@
 F 0 "C26" H 9790 3821 50  0000 L CNN
 F 1 "10uf_CH0" H 9725 3650 50  0000 L CNN
-F 2 "Capacitor_SMD:C_0805_2012Metric" H 9713 3625 50  0001 C CNN
+F 2 "Capacitor_THT:CP_Radial_D5.0mm_P2.00mm" H 9713 3625 50  0001 C CNN
 F 3 "~" H 9675 3775 50  0001 C CNN
 	1    9675 3775
@@
 F 0 "C4" V 5950 3150 50  0000 L CNN
 F 1 "10uf" V 6125 3075 50  0000 L CNN
-F 2 "Capacitor_SMD:C_0805_2012Metric" H 6038 2950 50  0001 C CNN
+F 2 "Capacitor_THT:CP_Radial_D5.0mm_P2.00mm" H 6038 2950 50  0001 C CNN
 F 3 "~" H 6000 3100 50  0001 C CNN
 	1    6000 3100
@@
 F 0 "C5" V 7300 1200 50  0000 L CNN
 F 1 "10uf" V 7475 1125 50  0000 L CNN
-F 2 "Capacitor_SMD:C_0805_2012Metric" H 7388 1000 50  0001 C CNN
+F 2 "Capacitor_THT:CP_Radial_D5.0mm_P2.00mm" H 7388 1000 50  0001 C CNN
 F 3 "~" H 7350 1150 50  0001 C CNN
 	1    7350 1150

Commit message: Cambios varios, Version 1 funcional
Parts:
- removed J4: Conn_02x06_Male_Pmod_Spartan6, Connector_PinHeader_2.54mm:PinHeader_2x06_P2.54mm_Horizontal, symbol Connector_Generic:Conn_02x06_Top_Bottom
- added J2, J3: Conn_01x06_Male, Connector_PinHeader_2.54mm:PinHeader_1x06_P2.54mm_Vertical, symbol Connector:Conn_01x06_Male
- C15: footprint Capacitor_SMD:C_0805_2012Metric -> Capacitor_SMD:C_0603_1608Metric
- C3: value 0.1uF -> 100nF
Connections:
- net ALARM: now also J3.5 (Pin_5)
- net CS: now also J2.6 (Pin_6)
- net GNDD: now also J2.2 (Pin_2), J3.2 (Pin_2)
- net RST-PD: now also J3.6 (Pin_6)
- net SCLK: now also J2.5 (Pin_5)
- net SDI: now also J2.3 (Pin_3)
- net SDO: now also J2.4 (Pin_4)
- net VDD: now also J2.1 (Pin_1), J3.1 (Pin_1)
Changed lines of the file:
@@
 EESchema Schematic File Version 4
-LIBS:PCB_ADS8694-cache
 EELAYER 29 0
 EELAYER END
@@
 $EndDescr
 $Comp
-L Connector_Generic:Conn_02x06_Top_Bottom J4
-U 1 1 5CCB59D8
-P 5100 1175
-F 0 "J4" H 5150 1592 50  0000 C CNN
-F 1 "Conn_02x06_Male_Pmod_Spartan6" H 5150 1501 50  0000 C CNN
-F 2 "Connector_PinHeader_2.54mm:PinHeader_2x06_P2.54mm_Horizontal" H 5100 1175 50  0001 C CNN
-F 3 "~" H 5100 1175 50  0001 C CNN
-	1    5100 1175
-	1    0    0    -1
-$EndComp
-$Comp
 L Regulator_Linear:LM7805_TO220 U1
 U 1 1 5CCB832F
@@
 P 2500 1200
 F 0 "C3" H 2618 1246 50  0000 L CNN
-F 1 "0.1uF" H 2618 1155 50  0000 L CNN
+F 1 "100nF" H 2618 1155 50  0000 L CNN
 F 2 "Capacitor_THT:C_Disc_D5.0mm_W2.5mm_P5.00mm" H 2538 1050 50  0001 C CNN
 F 3 "~" H 2500 1200 50  0001 C CNN
@@
 Wire Notes Line
 	950  650  950  1800
-Text GLabel 5400 1175 2    50   Input ~ 10
-SCLK
-Text GLabel 5400 975  2    50   Input ~ 10
-SDO
-Text GLabel 5400 1275 2    50   Input ~ 10
-SDI
-Wire Notes Line
-	6200 650  4150 650
 Text Notes 1400 2700 0    50   ~ 10
 FUENTE DE CC EXTERNA, +-VCC
@@
 Wire Wire Line
 	5250 3700 4600 3700
-NoConn ~ 4900 1475
-NoConn ~ 5400 1075
-$Comp
-L power:GNDD #PWR0118
-U 1 1 5CD843B0
-P 4475 1200
-F 0 "#PWR0118" H 4475 950 50  0001 C CNN
-F 1 "GNDD" H 4479 1045 50  0000 C CNN
-F 2 "" H 4475 1200 50  0001 C CNN
-F 3 "" H 4475 1200 50  0001 C CNN
-	1    4475 1200
-	1    0    0    -1
-$EndComp
 $Comp
 L power:GNDD #PWR0119
@@
 Text Notes 1275 4175 0    50   ~ 10
 CONECTORES DE ENTRADA DE SEÑAL
-$Comp
-L power:VDD #PWR0112
-U 1 1 5CD79A34
-P 4900 975
-F 0 "#PWR0112" H 4900 825 50  0001 C CNN
-F 1 "VDD" V 4918 1102 50  0000 L CNN
-F 2 "" H 4900 975 50  0001 C CNN
-F 3 "" H 4900 975 50  0001 C CNN
-	1    4900 975
-	0    -1   -1   0
-$EndComp
-$Comp
-L power:VDD #PWR0116
-U 1 1 5CD7F938
-P 4900 1075
-F 0 "#PWR0116" H 4900 925 50  0001 C CNN
-F 1 "VDD" V 4917 1203 50  0000 L CNN
-F 2 "" H 4900 1075 50  0001 C CNN
-F 3 "" H 4900 1075 50  0001 C CNN
-	1    4900 1075
-	0    -1   -1   0
-$EndComp
 $Comp
 L power:PWR_FLAG #FLG0101
@@
 F 0 "C15" H 3975 3175 50  0000 L CNN
 F 1 "1uf" H 4200 3350 50  0000 L CNN
-F 2 "Capacitor_SMD:C_0805_2012Metric" H 4213 3100 50  0001 C CNN
+F 2 "Capacitor_SMD:C_0603_1608Metric" H 4213 3100 50  0001 C CNN
 F 3 "~" H 4175 3250 50  0001 C CNN
 	1    4175 3250
@@
 Wire Wire Line
 	6825 4000 6250 4000
-Text GLabel 5400 1475 2    50   Input ~ 10
-RST-PD
-Text GLabel 4900 1375 0    50   Input ~ 10
-ALARM
-Text GLabel 5400 1375 2    50   Input ~ 10
-CS
 $Comp
 L ads8694_vers2:ADS8694_Vers2 U4
@@
 	5800 5900 5700 5900
 Wire Notes Line
-	4150 650  4150 1750
-Wire Notes Line
-	4150 1750 6200 1750
+	4100 650  4100 1750
 Wire Notes Line
 	6200 1750 6200 650
@@
 	5600 5900 5700 5900
 Connection ~ 5700 5900
-Wire Wire Line
-	4900 1275 4825 1275
-Wire Wire Line
-	4825 1275 4825 1175
-Connection ~ 4825 1175
-Wire Wire Line
-	4825 1175 4900 1175
-Wire Wire Line
-	4475 1200 4475 1175
-Wire Wire Line
-	4475 1175 4825 1175
+$Comp
+L Connector:Conn_01x06_Male J2
+U 1 1 5CF71E08
+P 4350 1125
+F 0 "J2" H 4458 1506 50  0000 C CNN
+F 1 "Conn_01x06_Male" H 4458 1415 50  0000 C CNN
+F 2 "Connector_PinHeader_2.54mm:PinHeader_1x06_P2.54mm_Vertical" H 4350 1125 50  0001 C CNN
+F 3 "~" H 4350 1125 50  0001 C CNN
+	1    4350 1125
+	1    0    0    -1
+$EndComp
+$Comp
+L Connector:Conn_01x06_Male J3
+U 1 1 5CF72D62
+P 5450 1125
+F 0 "J3" H 5558 1506 50  0000 C CNN
+F 1 "Conn_01x06_Male" H 5558 1415 50  0000 C CNN
+F 2 "Connector_PinHeader_2.54mm:PinHeader_1x06_P2.54mm_Vertical" H 5450 1125 50  0001 C CNN
+F 3 "~" H 5450 1125 50  0001 C CNN
+	1    5450 1125
+	1    0    0    -1
+$EndComp
+$Comp
+L power:VDD #PWR01
+U 1 1 5CF73629
+P 4550 925
+F 0 "#PWR01" H 4550 775 50  0001 C CNN
+F 1 "VDD" V 4568 1052 50  0000 L CNN
+F 2 "" H 4550 925 50  0001 C CNN
+F 3 "" H 4550 925 50  0001 C CNN
+	1    4550 925
+	0    1    1    0
+$EndComp
+$Comp
+L power:VDD #PWR036
+U 1 1 5CF783CD
+P 5650 925
+F 0 "#PWR036" H 5650 775 50  0001 C CNN
+F 1 "VDD" V 5668 1052 50  0000 L CNN
+F 2 "" H 5650 925 50  0001 C CNN
+F 3 "" H 5650 925 50  0001 C CNN
+	1    5650 925
+	0    1    1    0
+$EndComp
+$Comp
+L power:GNDD #PWR07
+U 1 1 5CF786F3
+P 5000 1025
+F 0 "#PWR07" H 5000 775 50  0001 C CNN
+F 1 "GNDD" H 5004 870 50  0000 C CNN
+F 2 "" H 5000 1025 50  0001 C CNN
+F 3 "" H 5000 1025 50  0001 C CNN
+	1    5000 1025
+	1    0    0    -1
+$EndComp
+$Comp
+L power:GNDD #PWR037
+U 1 1 5CF7E8E9
+P 6075 1025
+F 0 "#PWR037" H 6075 775 50  0001 C CNN
+F 1 "GNDD" H 6079 870 50  0000 C CNN
+F 2 "" H 6075 1025 50  0001 C CNN
+F 3 "" H 6075 1025 50  0001 C CNN
+	1    6075 1025
+	1    0    0    -1
+$EndComp
+Wire Wire Line
+	6075 1025 5650 1025
+Text GLabel 5650 1325 2    50   Input ~ 10
+ALARM
+Wire Wire Line
+	4550 1025 5000 1025
+NoConn ~ 5650 1125
+Text GLabel 4550 1225 2    50   Input ~ 10
+SDO
+NoConn ~ 5650 1225
+Text GLabel 4550 1325 2    50   Input ~ 10
+SCLK
+Text GLabel 4550 1125 2    50   Input ~ 10
+SDI
+Text GLabel 4550 1425 2    50   Input ~ 10
+CS
+Text GLabel 5650 1425 2    50   Input ~ 10
+RST-PD
+Wire Notes Line
+	4100 1750 6200 1750
+Wire Notes Line
+	4100 650  6200 650
 $EndSCHEMATC

Commit message: version finalizada
Changed lines of the file:
@@
 P 5850 3100
 F 0 "#PWR09" H 5850 2950 50  0001 C CNN
-F 1 "VDD" H 5867 3273 50  0000 C CNN
+F 1 "VDD" H 5900 3250 50  0000 C CNN
 F 2 "" H 5850 3100 50  0001 C CNN
 F 3 "" H 5850 3100 50  0001 C CNN
@@
 U 1 1 5CE32CBF
 P 5750 4500
-F 0 "U4" H 5750 5981 50  0000 C CNN
-F 1 "ADS8694_Vers2" H 5750 5890 50  0000 C CNN
+F 0 "U4" H 5725 4525 50  0000 C CNN
+F 1 "ADS8694_Vers2" H 5725 4425 50  0000 C CNN
 F 2 "Package_SO:TSSOP-38_4.4x9.7mm_P0.5mm" H 5750 4500 50  0001 C CNN
 F 3 "http://www.ti.com/lit/ds/symlink/ads8694.pdf" H 6700 5800 50  0001 C CNN
