File: Kicad_Design/PCB_ADS8694/PCB_ADS8694.kicad_pcb (KiCad board)
At the start: 2 copper layers, 47 parts, among them J1 Screw_Terminal_01x03_Alimenta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, J2 Conn_01x06_Male, J3 Conn_01x06_Male, J5 Screw_Terminal_01x02_CH3, J6 Screw_Terminal_01x02_CH2, J7 Screw_Terminal_01x02_CH1, J8 Screw_Terminal_01x02_CH0, U1 LM7805_TO220, U2 AD8221, U3 AD8221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

Commit message: Se agrega DCP01B, alimentado por lm7805. LA alimentacion de la placa debe ser mayor a 7V
Parts:
- added C11: CP, Capacitor_THT:CP_Radial_D5.0mm_P2.00mm, B.Cu at (170.3, 122.8)
- added C20: CP, Capacitor_THT:CP_Radial_D5.0mm_P2.00mm, B.Cu at (143.1, 129.9)
- added C30: CP, Capacitor_THT:CP_Radial_D5.0mm_P2.00mm, B.Cu at (143.2, 123.0)
- added U7: DCP01B, Package_DIP:DIP-14_W7.62mm, B.Cu at (163.8, 127.5)
- moved J1 16.0 mm to (161.1, 138.2)
- moved C1 7.83 mm to (170.0, 132.3)
Connections:
- C1 pad 1: VCC -> V_PWR
- J1 pad 2: VSS -> (no net)
- J1 pad 3: VCC -> V_PWR
- U1 pad 1: VCC -> V_PWR
Routing:
- net V_PWR: track 0.00 -> 34.3 mm
- net AVDD: track 55.7 -> 85.1 mm
- net VCC: track 237.6 -> 231.9 mm
- net VSS: track 198.7 -> 196.7 mm
